File: Hardware/SparkFun_Qwiic_Formaldehyde_Sensor_SFA40.kicad_pcb (KiCad board)
At the start: 2 copper layers, 25.4 x 25.4 mm, 39 parts, among them J1 Qwiic_RA, J2 Qwiic_RA, J3 Conn_01x06, U3 SFA40

Commit message: Design Review Changes
Parts:
- removed kibuzzard-689A66E9: G***, kibuzzard-689A66E9
- removed kibuzzard-689A6721: G***, kibuzzard-689A6721
- removed kibuzzard-6A1DC0D7 (x2): G***, kibuzzard-6A1DC0D7
- removed kibuzzard-6A1DC129: G***, kibuzzard-6A1DC129
- added G***: LOGO, SparkFun-Aesthetic:SparkFun_Logo_NoFlame_10mm, F.Cu at (135.9, 87.0)
- added kibuzzard-6A233140: G***, kibuzzard-6A233140, F.Cu at (136.0, 90.2)
- added kibuzzard-6A23318A: G***, kibuzzard-6A23318A, B.Cu at (134.7, 107.3)
- added kibuzzard-6A233190: G***, kibuzzard-6A233190, F.Cu at (134.7, 107.3)
- added kibuzzard-6A233774: G***, kibuzzard-6A233774, B.Cu at (133.4, 98.4)
- added kibuzzard-6A233784: G***, kibuzzard-6A233784, B.Cu at (133.4, 96.2)
- added kibuzzard-6A23378A: G***, kibuzzard-6A23378A, B.Cu at (132.6, 96.8)
- Ref**: moved to F.Cu
- moved G*** 21.6 mm to (127.4, 92.1)
- moved C5 11.4 mm to (129.9, 104.1), turned to -90 degrees
- moved R4 4.41 mm to (142.0, 106.7), turned to 180 degrees
- moved R5 4.41 mm to (129.9, 106.7), turned to 0 degrees
- moved U3 2.54 mm to (136.0, 98.1)
- moved kibuzzard-6A172007 2.22 mm to (135.9, 88.9)
- moved Ref** 1.37 mm to (144.9, 104.1), turned to 0 degrees
- moved G*** 0.32 mm to (136.0, 89.2)
Routing:
- net Net-(JP2-C): track 4.88 -> 9.00 mm
- net 3.3V: track 50.4 -> 47.5 mm
- net Net-(JP2-A): track 4.59 -> 7.42 mm
- net SDA: track 49.1 -> 51.8 mm
- net SCL: track 33.9 -> 35.6 mm
- net GND: track 4.99 -> 3.61 mm, vias 21 -> 20

Commit message: Rolls version to v10
Other:
- board text added: "v10"
- board text removed: "v01"
