File: Hardware/SparkFun_Qwiic_Formaldehyde_Sensor_SFA40.kicad_sch (KiCad schematic)
At the start: 23 parts, among them J1 Qwiic_RA, J2 Qwiic_RA, J3 Conn_01x06, U3 SFA40

Commit message: Design Review Changes
Parts:
- U3: PROD_ID (none) -> IC-28735
Other:
- note removed: "See table below for alternate addresses"
- moved on the sheet: D1, J1, J2, J3, R3, R4, R5
